File: hardware/BRD161001/BRD161001.brd (EAGLE design)
At the start: 57 x 33 mm, 43 parts, among them CN1 XH, CN2 JST XH, CN3 30306-6002HB, Q1 FDV301, Q2 DMP2035, Q3 FDV301, Q4 FDV301, U1 ATTINY44A-SSU, U2 TC4427AEOA, U3 TC4427AEOA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

Commit message: R1 of the hardware design
Signed-off-by: Christoph Tack <prog.send@gmail.com>
Parts:
- removed C1: 100u, lieBtrau:CA_POL_10X10
- removed C2, C8: 1U, lieBtrau:CA_1206
- removed D10, D3, D4, D5, D6, D7, D8, D9: MBRS240LT3G, lieBtrau:DI_DO214AA_SMB
- removed D2: BAT46W, lieBtrau:SOD323_ST
- removed DRILEGEND: (no value), drilegend:DRILEGEND
- removed U$1: FR_FRAME_A4, lieBtrau:FR_FRAME_A5
- removed U2, U3: TC4427AEOA, lieBtrau:SC_SO08
- added FR1: FR_FRAME_A4A5, lieBtrau:FR_FRAME_A5
- added HY1: SX1308 MODULE, lieBtrau:HY_SX1308
- added Q10, Q5, Q6, Q9: BC857, lieBtrau:SC_SOT23
- added Q11: DMP2035, lieBtrau:SC_SOT23
- added Q12: FDV301, lieBtrau:SC_SOT23
- added Q7, Q8: BC847, lieBtrau:SC_SOT23
- added R13, R14: 10K, lieBtrau:RE_1206
- added R15, R16: 390K, lieBtrau:RE_1206
- Q2: value DMP2035 -> BC847
- Q4: value FDV301 -> BC847
- R10, R11: value 4K7 -> 100K
- R2: value 1M -> 1M5
- R5: value 330K -> 390K
- R6: value 330K -> 100K
- R7: value 1M -> 100K
- R8, R9: value 4K7 -> 10K
- moved CN1 104.2 mm to (4.45, 3.94), turned to 180 degrees
- moved D1 86.6 mm to (18.0, 5.27)
- moved Q1 72.9 mm to (13.8, 4.09)
- moved R5 72.7 mm to (10.5, 4.10)
- moved CN2 70.5 mm to (39.6, 25.8)
- moved R4 69.8 mm to (17.6, 9.97)
- moved C3 68.7 mm to (11.9, 9.35), turned to 270 degrees
- moved C5 68.1 mm to (5.25, 31.7), turned to 180 degrees
- moved R8 66.6 mm to (20.1, 25.5)
- moved R9 65.8 mm to (20.1, 22.2), turned to 180 degrees
- moved Q3 65.6 mm to (18.0, 13.1)
- moved R2 65.4 mm to (14.0, 8.50), turned to 90 degrees
- moved R3 62.1 mm to (5.15, 23.1)
- moved C4 62.1 mm to (3.42, 29.6)
- moved X1 62.1 mm to (6.31, 28.6)
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Connections:
- new net N$26: R13.1, U1.13
- new net N$27: Q12.1, U1.6
- new net N$28: Q12.3, R16.1
- new net N$29: HY1.VIN, Q11.3
- new net N$8: CN2.4, Q4.3, Q5.3, R7.1
- net 3V3: no longer D2.C
- net GND: now also HY1.GND1, HY1.GND2, Q12.2, Q2.2, Q7.2, Q8.2; no longer C1.-, C2.2, C8.2, D10.A, D7.A, D8.A, D9.A, U2.3, U3.3
- net N$10: now also CN2.3, Q2.3, Q6.3, R6.1; no longer Q4.1, U1.6
- net N$11: now also Q2.1, R8.2; no longer C2.1, C8.1, D3.C, D4.C, D5.C, D6.C, Q2.3, U2.6, U3.6
- net N$12: now also Q4.1, R9.1; no longer R8.1, U1.13
- net N$13: now also HY1.OUT, Q10.2, Q9.2; no longer R9.1, U1.12
- net N$14: now also R9.2, U1.10; no longer R10.1, U1.11
- net N$15: now also R8.1, U1.11; no longer R11.1, U1.10
- net N$16: now also Q9.1, R10.2; no longer R8.2, U2.2
- net N$17: now also Q10.1, R11.2; no longer R9.2, U2.4
- net N$18: now also Q7.1, R13.2; no longer R10.2, U3.2
- net N$19: now also Q8.1, R14.1; no longer R11.2, U3.4
- net N$2: now also D1.C, Q11.2, Q3.3, Q5.2, Q6.2, R15.2, R4.2; no longer Q2.1, R6.1, R7.2
- net N$20: now also R14.2, U1.12; no longer CN2.1, D3.A, D7.C, U2.7
- net N$21: now also Q11.1, R15.1, R16.2; no longer CN2.2, D4.A, D8.C, U2.5
- net N$22: now also CN2.2, Q8.3, Q9.3, R11.1; no longer CN2.3, D5.A, D9.C, U3.7
- net N$23: now also CN2.1, Q10.3, Q7.3, R10.1; no longer CN2.4, D10.C, D6.A, U3.5
- net N$3: now also Q5.1; no longer C1.+, D1.C, Q2.2, Q3.3, R4.2
- net N$5: now also Q6.1, R7.2; no longer Q4.3, R7.1
- net RST: no longer D2.A
Routing:
- net N$11: track 42.6 -> 5.77 mm
- net N$2: track 4.55 -> 40.2 mm, vias 0 -> 3
- net N$13: track 4.42 -> 37.6 mm, vias 0 -> 2
- net 3V3: track 79.5 -> 49.4 mm
- net N$20: track 29.9 -> 4.40 mm
- net N$21: track 28.5 -> 6.19 mm
- net N$3: track 27.9 -> 7.08 mm
- net N$23: track 35.3 -> 17.2 mm
- net N$8: track 0.00 -> 17.1 mm
- net N$27: track 0.00 -> 10.8 mm
- net N$22: track 28.1 -> 18.2 mm
- net N$29: track 0.00 -> 8.74 mm
- net N$4: track 4.74 -> 12.0 mm
- net N$1: track 7.45 -> 14.3 mm
- net GND: track 44.7 -> 38.9 mm
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Other:
- board size 57 x 33 mm -> 43.5 x 34 mm
- board text added: "BRD1611001/1"

Commit message: working on R2 of PCB
Signed-off-by: Christoph Tack <prog.send@gmail.com>
Parts:
- moved CN2 1.22 mm to (40.8, 25.8)
- moved CN1 0.06 mm to (4.40, 3.90), turned to 0 degrees
Routing:
- net RST: track 13.4 -> 7.09 mm
- net N$1: track 14.3 -> 16.9 mm
- net GND: track 38.9 -> 40.3 mm
- net N$10: track 17.5 -> 18.7 mm
- net N$8: track 17.1 -> 18.3 mm
- net N$23: track 17.2 -> 18.4 mm
- net N$22: track 18.2 -> 19.4 mm
- net N$13: track 37.6 -> 38.6 mm
- net N$2: track 40.2 -> 41.0 mm

Commit message: R2 of BRD161001
Signed-off-by: Christoph Tack <prog.send@gmail.com>
Parts:
- removed FR1: FR_FRAME_A4A5, lieBtrau:FR_FRAME_A5
- added U$2: (no value), lieBtrau:FR_FRAME_A5
Routing:
- net RST: track 7.09 -> 13.4 mm
Other:
- board text added: "BRD1611001/2"
- board text removed: "BRD1611001/1"
